Commit message: Progress so far

File: urdf/Xarm.urdf (robot description, URDF)
Before this commit: robot Jahwin_arm, 3 links, 2 joints
Joints:
- removed joint joint_name
- removed joint two_one
- added joint base_to_link1: type revolute, parent base_link, child link1, origin xyz=0 0 0.356 rpy=0 0 0, axis 0 0 1, limit lower=-3.1416 upper=3.1416 effort=10 velocity=1.0
- added joint link1_to_link2: type revolute, parent link1, child link2, origin xyz=0 0 0 rpy=0 0 0, axis 0 1 0, limit lower=-3.1416 upper=3.1416 effort=20 velocity=0.6

Commit message: Progress so far

File: urdf/Xarm.urdf (robot description, URDF)
Before this commit: robot Jahwin_arm, 3 links, 2 joints
Links:
- added link link3; visual mesh filename=package://xarm_description/meshes/link3.stl scale=1.0 1.0 1.0
- added link link4; visual mesh filename=package://xarm_description/meshes/link4.stl scale=1.0 1.0 1.0
- added link link5; visual mesh filename=package://xarm_description/meshes/link5.stl scale=1.0 1.0 1.0
- added link link6; visual mesh filename=package://xarm_description/meshes/link6.stl scale=1.0 1.0 1.0
Joints:
- added joint link2_to_link3: type revolute, parent link2, child link3, origin xyz=0 0 0.4 rpy=0 0 0, axis 0 1 0, limit lower=-3.1416 upper=3.1416 effort=20 velocity=0.6
- added joint link3_to_link4: type revolute, parent link3, child link4, origin xyz=0.15 0 -0.15 rpy=0 0 0, axis 0 0 1, limit lower=-3.1416 upper=3.1416 effort=20 velocity=0.6
- added joint link4_to_link5: type revolute, parent link4, child link5, origin xyz=0 0 -0.265 rpy=0 0 0, axis 0 0 1, limit lower=-3.1416 upper=3.1416 effort=20 velocity=0.6
- added joint link5_to_link6: type revolute, parent link5, child link6, origin xyz=0 0 0 rpy=0 0 0, axis 0 0 1, limit lower=-3.1416 upper=3.1416 effort=20 velocity=0.6

Commit message: Progress so far

File: urdf/Xarm.urdf (robot description, URDF)
Before this commit: robot Jahwin_arm, 7 links, 6 joints
Joints:
- joint link4_to_link5: axis 0 0 1 -> 0 1 0

Commit message: Progress so far

File: urdf/Xarm.urdf (robot description, URDF)
Before this commit: robot Jahwin_arm, 7 links, 6 joints
Links:
- link base_link: geometry collision mesh filename=package://xarm_description/meshes/link_base.stl scale=1.0 1.0 1.0; visual mesh filename=package://xarm_description/meshes/link_base.stl scale=1.0 1.0 1.0
- link link1: geometry collision mesh filename=package://xarm_description/meshes/link1.stl scale=1.0 1.0 1.0; visual mesh filename=package://xarm_description/meshes/link1.stl scale=1.0 1.0 1.0
- link link2: geometry collision mesh filename=package://xarm_description/meshes/link2.stl scale=1.0 1.0 1.0; visual mesh filename=package://xarm_description/meshes/link2.stl scale=1.0 1.0 1.0
- link link3: geometry collision mesh filename=package://xarm_description/meshes/link3.stl scale=1.0 1.0 1.0; visual mesh filename=package://xarm_description/meshes/link3.stl scale=1.0 1.0 1.0
- link link4: geometry collision mesh filename=package://xarm_description/meshes/link4.stl scale=1.0 1.0 1.0; visual mesh filename=package://xarm_description/meshes/link4.stl scale=1.0 1.0 1.0
- link link5: geometry collision mesh filename=package://xarm_description/meshes/link5.stl scale=1.0 1.0 1.0; visual mesh filename=package://xarm_description/meshes/link5.stl scale=1.0 1.0 1.0
- link link6: geometry collision mesh filename=package://xarm_description/meshes/link6.stl scale=1.0 1.0 1.0; visual mesh filename=package://xarm_description/meshes/link6.stl scale=1.0 1.0 1.0
